File: Board/quadcopter.brd (EAGLE design)
At the start: 60 x 60 mm, 56 parts, among them M1+ TPTP20SQ, M1- TPTP20SQ, M2+ TPTP20SQ, M2- TPTP20SQ, M3+ TPTP20SQ, M3- TPTP20SQ, M4+ TPTP20SQ, M4- TPTP20SQ, U2 LTC1844ES5-3.3TRMPBF, Y1 12MHZ

Commit message: Fix in Powersupply
0.1uF instead of 1uF for bypass capacitor
Parts:
- C3: value 1u -> 0.1u
Changed lines of the file:
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@@
 <attribute name="PROD_ID" value="RES-08296" x="13.15" y="8.25" size="1.778" layer="27" rot="R180" display="off"/>
 </element>
-<element name="C3" library="SparkFun-Capacitors" package="0603-CAP" value="1u" x="15.95" y="11.65" rot="R90">
+<element name="C3" library="SparkFun-Capacitors" package="0603-CAP" value="0.1u" x="15.95" y="11.65" rot="R90">
 <attribute name="PROD_ID" value="CAP-11015" x="15.95" y="11.65" size="1.778" layer="27" rot="R90" display="off"/>
 </element>
